File: pcb/pathfinder.kicad_pcb (KiCad board)
At the start: 2 copper layers, 10 parts, among them SW1 SW_Push, SW2 SW_Push, SW3 SW_Push, U1 XIAO-RP2040-DIP

Commit message: finished pcb and other small stuff
Parts:
- added  : LOGO, sonic:sonic_ring, F.Cu at (168.5, 75.5)
- added   : LOGO, sonic:sonic_ring, F.Cu at (150.5, 51.0)
- added   : LOGO, sonic:sonic_running, F.Cu at (149.0, 61.5)
- added   : LOGO, sonic:sonic_running, F.Cu at (220.0, 62.5)
- added  : LOGO, sonic:sonic_ring, F.Cu at (200.5, 29.0)
- added  : LOGO, sonic:sonic_ring, F.Cu at (160.5, 33.5)
- added  : LOGO, sonic:sonic_ring, F.Cu at (154.5, 49.5)
- added  : LOGO, sonic:sonic_ring, F.Cu at (171.0, 79.0)
- added  : LOGO, sonic:sonic_ring, F.Cu at (223.5, 55.0)
- added  : LOGO, sonic:sonic_ring, F.Cu at (219.0, 54.0)
- added  : LOGO, sonic:sonic_ring, F.Cu at (163.5, 30.0)
- added  : LOGO, sonic:sonic_ring, F.Cu at (168.0, 28.5)
- added  : LOGO, sonic:emeralds, F.Cu at (212.5, 45.5)
- added  : LOGO, sonic:sonic_ring, F.Cu at (151.5, 47.1)
- added  : LOGO, sonic:sonic_ring, F.Cu at (204.0, 31.0)
- added  : LOGO, sonic:sonic_ring, F.Cu at (198.0, 78.5)
- added  : LOGO, sonic:sonic_ring, F.Cu at (164.0, 76.0)
- added G***: LOGO, sonic:sonics_emerald_v2, B.Cu at (185.5, 57.5)
- SW1, SW2, SW3: footprint Button_Switch_Keyboard:SW_Cherry_MX_1.00u_PCB -> Seeed Studio XIAO Series Library:MX_KeySwitch 3D
- moved SW3 92.2 mm to (207.2, 56.8)
- moved R3 67.1 mm to (186.8, 59.8), turned to 180 degrees
- moved D3 66.6 mm to (203.5, 40.5), turned to 180 degrees
- moved SW2 63.2 mm to (186.6, 67.2)
- moved R1 63.0 mm to (181.7, 53.5)
- moved R2 63.0 mm to (181.7, 56.7)
- moved U1 58.6 mm to (183.5, 39.8)
- moved SW1 42.2 mm to (166.0, 56.9)
- moved D1 32.3 mm to (164.6, 40.6)
- moved D2 30.2 mm to (184.7, 85.3), turned to 180 degrees
Routing:
- net GND: track 0.00 -> 117.6 mm
- net Net-(U1-GPIO28/ADC2/A2): track 0.00 -> 43.8 mm, vias 0 -> 1
- net Net-(U1-GPIO26/ADC0/A0): track 0.00 -> 41.6 mm
- net Net-(U1-GPIO27/ADC1/A1): track 0.00 -> 38.0 mm
- net Net-(D2-PadA): track 0.00 -> 35.3 mm
- net Net-(D3-PadA): track 0.00 -> 25.7 mm
- net Net-(D1-PadA): track 0.00 -> 21.1 mm
- net led1: track 0.00 -> 19.7 mm
- net led0: track 0.00 -> 19.1 mm
- net led2: track 0.00 -> 19.1 mm
- net unconnected-(U1-VBUS-Pad14): track 0.00 -> 0.84 mm
- net unconnected-(U1-GPIO4/MISO-Pad10): track 0.00 -> 0.84 mm
- net unconnected-(U1-GPIO3/MOSI-Pad11): track 0.00 -> 0.84 mm
- net unconnected-(U1-GPIO2/SCK-Pad9): track 0.00 -> 0.84 mm
- net unconnected-(U1-GPIO1/RX-Pad8): track 0.00 -> 0.84 mm
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Other:
- board outline added: 88 x 67 mm
