File: pcb/pathfinder.kicad_sch (KiCad schematic)
At the start: 1 part, among them U1 XIAO-RP2040-DIP

Commit message: stuff
Parts:
- added D1, D2, D3: led, led:LEDRD254W57D500H1070, symbol led:L08R5000Q1
- added R1, R2, R3: R, Resistor_THT:R_Axial_DIN0204_L3.6mm_D1.6mm_P5.08mm_Horizontal, symbol Device:R
- added SW1, SW2, SW3: SW_Push, Button_Switch_Keyboard:SW_Cherry_MX_1.00u_PCB, symbol Switch:SW_Push
- U1: footprint Module:MOUDLE14P-XIAO-DIP-SMD -> Seeed Studio XIAO Series Library:XIAO-RP2040-DIP
Connections:
- net at U1.1 (GPIO26/ADC0/A0): now also SW2.2
- net GND: now reaches U1.13 (GND)
- net GND: now also D1.C, D2.C, D3.C, SW1.1, SW2.1, SW3.1
- net at U1.2 (GPIO27/ADC1/A1): now also SW1.2
- net at U1.3 (GPIO28/ADC2/A2): now also SW3.2
- net led0: now reaches U1.4 (GPIO29/ADC3/A3)
- net led0: now also R1.2
- net led1: now reaches U1.5 (GPIO6/SDA)
- net led1: now also R2.2
- net led2: now reaches U1.6 (GPIO7/SCL)
- net led2: now also R3.2
- new net: D2.A, R2.1
- new net: D3.A, R3.1
- new net: D1.A, R1.1

Commit message: finished pcb and other small stuff
Parts:
- SW1, SW2, SW3: footprint Button_Switch_Keyboard:SW_Cherry_MX_1.00u_PCB -> Seeed Studio XIAO Series Library:MX_KeySwitch 3D
Changed lines of the file:
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@@
 			)
 		)
-		(property "Footprint" "Button_Switch_Keyboard:SW_Cherry_MX_1.00u_PCB"
+		(property "Footprint" "Seeed Studio XIAO Series Library:MX_KeySwitch 3D"
 			(at 114.3 113.03 0)
 			(effects
@@
 			)
 		)
-		(property "Footprint" "Button_Switch_Keyboard:SW_Cherry_MX_1.00u_PCB"
+		(property "Footprint" "Seeed Studio XIAO Series Library:MX_KeySwitch 3D"
 			(at 114.3 105.41 0)
 			(effects
@@
 			)
 		)
-		(property "Footprint" "Button_Switch_Keyboard:SW_Cherry_MX_1.00u_PCB"
+		(property "Footprint" "Seeed Studio XIAO Series Library:MX_KeySwitch 3D"
 			(at 114.3 109.22 0)
 			(effects
